File: PCB/MP3Player.kicad_pcb (KiCad board)
At the start: 2 copper layers, 30.5 x 60 mm, 4 parts, among them J1 Raspberry_Pi_4, SW1 RotaryEncoder_Switch, SW2 SW_Push, SW3 SW_Push

Commit message: drill holes
Parts:
- added H1: MountingHole, MountingHole:MountingHole_2.2mm_M2, F.Cu at (156.0, 51.0)
- added H2: MountingHole, MountingHole:MountingHole_2.2mm_M2, F.Cu at (156.0, 105.0)
- moved SW1 2.00 mm to (140.5, 94.0)
Other:
- board size 30.5 x 60 mm -> 30.5 x 59 mm
Changed lines of the file:
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@@
 			(outputformat 1)
 			(mirror no)
-			(drillshape 1)
+			(drillshape 0)
 			(scaleselection 1)
-			(outputdirectory "")
+			(outputdirectory "E:/PYPROJ/odo/mp3/PCB/Production")
 		)
 	)
@@
 	(net 30 "unconnected-(J1-ID_SD_I2C0{slash}GPIO00-Pad27)")
 	(net 31 "unconnected-(J1-GPIO20{slash}SPI1_MOSI{slash}PCM_DIN{slash}PWM1-Pad38)")
+	(footprint "MountingHole:MountingHole_2.2mm_M2"
+		(layer "F.Cu")
+		(at 156 105)
+		(descr "Mounting Hole 2.2mm, no annular, M2")
+		(tags "mounting hole 2.2mm no annular m2")
+		(property "Reference" "H2"
+			(at 0 -3.2 0)
+			(layer "F.SilkS")
+			(effects
+				(font
+					(size 1 1)
+					(thickness 0.15)
+				)
+			)
+		)
+		(property "Value" "MountingHole"
+			(at 0 3.2 0)
+			(layer "F.Fab")
+			(effects
+				(font
+					(size 1 1)
+					(thickness 0.15)
+				)
+			)
+		)
+		(property "Datasheet" ""
+			(at 0 0 0)
+			(unlocked yes)
+			(layer "F.Fab")
+			(hide yes)
+			(effects
+				(font
+					(size 1.27 1.27)
+					(thickness 0.15)
+				)
+			)
+		)
+		(property "Description" "Mounting Hole without connection"
+			(at 0 0 0)
+			(unlocked yes)
+			(layer "F.Fab")
+			(hide yes)
+			(effects
+				(font
+					(size 1.27 1.27)
+					(thickness 0.15)
+				)
+			)
+		)
+		(property ki_fp_filters "MountingHole*")
+		(sheetname "/")
+		(sheetfile "MP3Player.kicad_sch")
+		(attr exclude_from_pos_files exclude_from_bom)
+		(fp_circle
+			(center 0 0)
+			(end 2.2 0)
+			(stroke
+				(width 0.15)
+				(type solid)
+			)
+			(fill no)
+			(layer "Cmts.User")
+		)
+		(fp_circle
+			(center 0 0)
+			(end 2.45 0)
+			(stroke
+				(width 0.05)
+				(type solid)
+			)
+			(fill no)
+			(layer "F.CrtYd")
+		)
+		(fp_text user "${REFERENCE}"
+			(at 0 0 0)
+			(layer "F.Fab")
+			(effects
+				(font
+					(size 1 1)
+					(thickness 0.15)
+				)
+			)
+		)
+		(pad "" np_thru_hole circle
+			(at 0 0)
+			(size 2.2 2.2)
+			(drill 2.2)
+			(layers "*.Cu" "*.Mask")
+		)
+		(embedded_fonts no)
+	)
+	(footprint "MountingHole:MountingHole_2.2mm_M2"
+		(layer "F.Cu")
+		(at 156 51)
+		(descr "Mounting Hole 2.2mm, no annular, M2")
+		(tags "mounting hole 2.2mm no annular m2")
+		(property "Reference" "H1"
+			(at 0 -3.2 0)
+			(layer "F.SilkS")
+			(effects
+				(font
+					(size 1 1)
+					(thickness 0.15)
+				)
+			)
+		)
+		(property "Value" "MountingHole"
+			(at 0 3.2 0)
+			(layer "F.Fab")
+			(effects
+				(font
+					(size 1 1)
+					(thickness 0.15)
+				)
+			)
+		)
+		(property "Datasheet" ""
+			(at 0 0 0)
+			(unlocked yes)
+			(layer "F.Fab")
+			(hide yes)
+			(effects
+				(font
+					(size 1.27 1.27)
+					(thickness 0.15)
+				)
+			)
+		)
+		(property "Description" "Mounting Hole without connection"
+			(at 0 0 0)
+			(unlocked yes)
+			(layer "F.Fab")
+			(hide yes)
+			(effects
+				(font
+					(size 1.27 1.27)
+					(thickness 0.15)
+				)
+			)
+		)
+		(property ki_fp_filters "MountingHole*")
+		(sheetname "/")
+		(sheetfile "MP3Player.kicad_sch")
+		(attr exclude_from_pos_files exclude_from_bom)
+		(fp_circle
+			(center 0 0)
+			(end 2.2 0)
+			(stroke
+				(width 0.15)
+				(type solid)
+			)
+			(fill no)
+			(layer "Cmts.User")
+		)
+		(fp_circle
+			(center 0 0)
+			(end 2.45 0)
+			(stroke
+				(width 0.05)
+				(type solid)
+			)
+			(fill no)
+			(layer "F.CrtYd")
+		)
+		(fp_text user "${REFERENCE}"
+			(at 0 0 0)
+			(layer "F.Fab")
+			(effects
+				(font
+					(size 1 1)
+					(thickness 0.15)
+				)
+			)
+		)
+		(pad "" np_thru_hole circle
+			(at 0 0)
+			(size 2.2 2.2)
+			(drill 2.2)
+			(layers "*.Cu" "*.Mask")
+		)
+		(embedded_fonts no)
+	)
 	(footprint "Connector_PinSocket_2.54mm:PinSocket_2x20_P2.54mm_Vertical"
 		(layer "F.Cu")
@@
 	(footprint "Rotary_Encoder:RotaryEncoder_Alps_EC11E-Switch_Vertical_H20mm_MountingHoles"
 		(layer "F.Cu")
-		(at 140.5 96)
+		(at 140.5 94)
 		(descr "Alps rotary encoder, EC12E... with switch, vertical shaft, https://www.lcsc.com/datasheet/lcsc_datasheet_2410010003_ALPSALPINE-EC11E09444A8_C1322538.pdf")
 		(tags "rotary encoder")
@@
 	)
 	(gr_line
-		(start 158.5 108.5)
+		(start 136.5 104.5)
+		(end 136.5 107.5)
+		(stroke
+			(width 0.05)
+			(type default)
+		)
+		(layer "Edge.Cuts")
+	)
+	(gr_line
+		(start 158.5 107.5)
 		(end 158.5 48.5)
+		(stroke
+			(width 0.05)
+			(type default)
+		)
+		(layer "Edge.Cuts")
+	)
+	(gr_line
+		(start 158.5 107.5)
+		(end 136.5 107.5)
 		(stroke
 			(width 0.05)
@@
 	)
 	(gr_line
-		(start 136.5 108.5)
-		(end 158.5 108.5)
-		(stroke
-			(width 0.05)
-			(type default)
-		)
-		(layer "Edge.Cuts")
-	)
-	(gr_line
 		(start 138 48.5)
 		(end 136.5 48.5)
@@
 	)
 	(gr_line
+		(start 154 103.5)
+		(end 158.5 107.5)
+		(stroke
+			(width 0.05)
+			(type default)
+		)
+		(layer "Edge.Cuts")
+	)
+	(gr_line
 		(start 158.5 48.5)
 		(end 138 48.5)
 		(stroke
 			(width 0.05)
-			(type default)
-		)
-		(layer "Edge.Cuts")
-	)
-	(gr_line
-		(start 136.5 104.5)
-		(end 136.5 108.5)
-		(stroke
-			(width 0.05)

Commit message: aaaaaa
Parts:
- moved H2 40.2 mm to (170.5, 142.5)
- moved SW1 37.4 mm to (151.6, 129.7)
- moved J1 35.1 mm to (143.5, 87.4)
- moved SW3 34.8 mm to (161.5, 107.3)
- moved SW2 34.0 mm to (161.5, 87.6)
- moved H1 32.4 mm to (170.5, 80.0)
Routing:
- net Net-(J1-3V3-Pad1): track 0.00 -> 37.5 mm
- net Net-(J1-GND-Pad14): track 91.9 -> 125.8 mm
- net Net-(J1-GPCLK1/GPIO05): track 31.3 -> 27.5 mm
- net Net-(J1-5V-Pad2): track 0.00 -> 2.54 mm
- net Net-(J1-GPCLK2/GPIO06): track 43.8 -> 45.3 mm
- net Net-(J1-GPIO26/SDIO_DAT2): track 32.4 -> 33.3 mm
Other:
- board size 30.5 x 59 mm -> 36 x 72 mm
